File: so16_breakout/main.brd (EAGLE design)
At the start: 27.6 x 30.5 mm, 5 parts

Commit message: [ update ] so16_breakout
Parts:
- removed JP3, JP4: (no value), SparkFun:1X04
- JP1, JP2: device SparkFun:1X04 -> SparkFun:1X08_LONGPADS
- moved JP2 22.9 mm to (5.08, 3.81)
- moved JP1 10.2 mm to (5.08, 26.7)
Connections:
- net N$1: now also JP1.8; no longer JP1.4
- net N$10: now also JP2.7; no longer JP3.3
- net N$11: now also JP2.6; no longer JP3.2
- net N$12: now also JP2.5; no longer JP3.1
- net N$13: now also JP2.4; no longer JP4.4
- net N$14: now also JP2.3; no longer JP4.3
- net N$15: now also JP2.2; no longer JP4.2
- net N$16: now also JP2.1; no longer JP4.1
- net N$2: now also JP1.7; no longer JP1.3
- net N$3: now also JP1.6; no longer JP1.2
- net N$4: now also JP1.5; no longer JP1.1
- net N$5: now also JP1.4; no longer JP2.4
- net N$6: now also JP1.3; no longer JP2.3
- net N$7: now also JP1.2; no longer JP2.2
- net N$8: now also JP1.1; no longer JP2.1
- net N$9: now also JP2.8; no longer JP3.4
Routing:
- net N$9: track 11.5 -> 14.9 mm
- net N$8: track 11.6 -> 14.9 mm
- net N$16: track 11.6 -> 14.9 mm
- net N$1: track 11.8 -> 14.9 mm
- net N$10: track 10.5 -> 13.0 mm
- net N$15: track 10.5 -> 13.0 mm
- net N$7: track 10.6 -> 13.0 mm
- net N$2: track 10.8 -> 13.0 mm
- net N$14: track 9.36 -> 11.1 mm
- net N$11: track 9.38 -> 11.1 mm
- net N$6: track 9.66 -> 11.1 mm
- net N$3: track 9.72 -> 11.1 mm
- net N$13: track 8.40 -> 9.18 mm
- net N$12: track 8.56 -> 9.18 mm
- net N$4: track 8.61 -> 9.18 mm
- added copper zone on layer 1, net N$17
Other:
- board size 27.6 x 30.5 mm -> 26.3 x 30.5 mm
